Commit message: feat:增加tcb710v、tcb710仿真

File: src/tl_description/urdf/tl_tcb710.urdf (robot description, URDF)
Before this commit: robot tcb710, 8 links, 7 joints
Links:
- link link3: mass 0.168577086504063 -> 0.168577225205791
- link link4: mass 0.145368322724393 -> 0.145368246128048
- link link5: mass 0.0899817886777035 -> 0.0899815381638705
- link link6: mass 0.0915266768417585 -> 0.0915266768417461
- link link7: mass 0.0756964619101267 -> 1.15874182567556
Joints:
- joint joint4: axis 0 0 1 -> 0 0 -1; origin xyz=0 -0.00515 0.16035 rpy=1.5708 0 -3.1416 -> xyz=0 -0.00515000000097151 0.160350000000103 rpy=1.5708 1.5708 0
- joint joint5: origin xyz=-0.16615 0 0.00515 rpy=1.5708 0 -1.5708 -> xyz=0 0.16615 -0.00515 rpy=-1.5708 0 0
- joint joint6: limit lower=-3.8386 upper=0.697 effort=0 velocity=0 -> lower=-3.8386 upper=0.6970 effort=0 velocity=0; origin xyz=0 0.00615 0.11335 rpy=-1.5708 0 0 -> xyz=0 0.00615 0.11335 rpy=-1.5708 1.5708 0
- joint joint7: origin xyz=0.10615 0 -0.00615 rpy=0 1.5708 0 -> xyz=0 -0.10615 -0.00615 rpy=1.5708 0 0
