Commit message: feat:添加705系列的moveit2+gazebo仿真

File: src/tl_moveit2_config/tl_tcb705_config/config/tl_tcb705.ros2_control.xacro (robot description, xacro)
@@ -1,5 +1,5 @@
 <?xml version="1.0"?>
 <robot xmlns:xacro="http://www.ros.org/wiki/xacro">
-    <xacro:macro name="tl_tcb710_ros2_control" params="name initial_positions_file">
+    <xacro:macro name="tl_tcb705_ros2_control" params="name initial_positions_file">
         <xacro:property name="initial_positions" value="${load_yaml(initial_positions_file)['initial_positions']}"/>
         <ros2_control name="${name}" type="system">

File: src/tl_moveit2_config/tl_tcb705f_config/config/tl_tcb705f.ros2_control.xacro (robot description, xacro)
@@ -1,5 +1,5 @@
 <?xml version="1.0"?>
 <robot xmlns:xacro="http://www.ros.org/wiki/xacro">
-    <xacro:macro name="tl_tcb710_ros2_control" params="name initial_positions_file">
+    <xacro:macro name="tl_tcb705f_ros2_control" params="name initial_positions_file">
         <xacro:property name="initial_positions" value="${load_yaml(initial_positions_file)['initial_positions']}"/>
         <ros2_control name="${name}" type="system">

File: src/tl_moveit2_config/tl_tcb705l_config/config/tl_tcb705l.ros2_control.xacro (robot description, xacro)
@@ -1,5 +1,5 @@
 <?xml version="1.0"?>
 <robot xmlns:xacro="http://www.ros.org/wiki/xacro">
-    <xacro:macro name="tl_tcb710_ros2_control" params="name initial_positions_file">
+    <xacro:macro name="tl_tcb705l_ros2_control" params="name initial_positions_file">
         <xacro:property name="initial_positions" value="${load_yaml(initial_positions_file)['initial_positions']}"/>
         <ros2_control name="${name}" type="system">

File: src/tl_moveit2_config/tl_tcb705lv_config/config/tl_tcb705lv.ros2_control.xacro (robot description, xacro)
@@ -1,5 +1,5 @@
 <?xml version="1.0"?>
 <robot xmlns:xacro="http://www.ros.org/wiki/xacro">
-    <xacro:macro name="tl_tcb710_ros2_control" params="name initial_positions_file">
+    <xacro:macro name="tl_tcb705lv_ros2_control" params="name initial_positions_file">
         <xacro:property name="initial_positions" value="${load_yaml(initial_positions_file)['initial_positions']}"/>
         <ros2_control name="${name}" type="system">

File: src/tl_moveit2_config/tl_tcb705v_config/config/tl_tcb705v.ros2_control.xacro (robot description, xacro)
@@ -1,5 +1,5 @@
 <?xml version="1.0"?>
 <robot xmlns:xacro="http://www.ros.org/wiki/xacro">
-    <xacro:macro name="tl_tcb710_ros2_control" params="name initial_positions_file">
+    <xacro:macro name="tl_tcb705v_ros2_control" params="name initial_positions_file">
         <xacro:property name="initial_positions" value="${load_yaml(initial_positions_file)['initial_positions']}"/>
         <ros2_control name="${name}" type="system">
