Commit message: feat:moveit2控制真实机械臂完成所有型号适配

File: src/tl_moveit2_config/tl_tcb605f_config/config/tl_tcb605f.ros2_control.xacro (robot description, xacro)
@@ -1,10 +1,19 @@
 <?xml version="1.0"?>
 <robot xmlns:xacro="http://www.ros.org/wiki/xacro">
-    <xacro:macro name="tl_tcb605f_ros2_control" params="name initial_positions_file">
+    <xacro:macro name="tl_tcb605f_ros2_control" params="name initial_positions_file use_real_hardware:=false">
         <xacro:property name="initial_positions" value="${xacro.load_yaml(initial_positions_file)['initial_positions']}"/>
         <ros2_control name="${name}" type="system">
             <hardware>
-                <!-- By default, set up controllers for simulation. This won't work on real hardware -->
-                <plugin>mock_components/GenericSystem</plugin>
+                <xacro:if value="${use_real_hardware}">
+                    <plugin>tl_hardware/TLHardwareInterface</plugin>
+                    <param name="joint_states_topic">/joint_states</param>
+                    <param name="servoj_topic">/tl_driver/set_servoj_pos</param>
+                    <param name="open_servoj_service">/tl_driver/open_servoj</param>
+                    <param name="close_servoj_service">/tl_driver/close_servoj</param>
+                    <param name="state_timeout_sec">1.0</param>
+                </xacro:if>
+                <xacro:unless value="${use_real_hardware}">
+                    <plugin>mock_components/GenericSystem</plugin>
+                </xacro:unless>
             </hardware>
             <joint name="joint1">

File: src/tl_moveit2_config/tl_tcb605f_config/config/tl_tcb605f.urdf.xacro (robot description, xacro)
@@ -2,8 +2,9 @@
 <robot xmlns:xacro="http://www.ros.org/wiki/xacro" name="tl_tcb605f">
     <xacro:arg name="initial_positions_file" default="initial_positions.yaml" />
+    <xacro:arg name="use_real_hardware" default="false" />
     <!-- Import tl_tcb605f urdf file -->
     <xacro:include filename="$(find tl_description)/urdf/tcb605f.urdf" />
     <!-- Import control_xacro -->
     <xacro:include filename="tl_tcb605f.ros2_control.xacro" />
-    <xacro:tl_tcb605f_ros2_control name="FakeSystem" initial_positions_file="$(arg initial_positions_file)"/>
+    <xacro:tl_tcb605f_ros2_control name="FakeSystem" initial_positions_file="$(arg initial_positions_file)" use_real_hardware="$(arg use_real_hardware)"/>
 </robot>

File: src/tl_moveit2_config/tl_tcb605l_config/config/tl_tcb605l.ros2_control.xacro (robot description, xacro)
@@ -1,10 +1,19 @@
 <?xml version="1.0"?>
 <robot xmlns:xacro="http://www.ros.org/wiki/xacro">
-    <xacro:macro name="tl_tcb605l_ros2_control" params="name initial_positions_file">
+    <xacro:macro name="tl_tcb605l_ros2_control" params="name initial_positions_file use_real_hardware:=false">
         <xacro:property name="initial_positions" value="${xacro.load_yaml(initial_positions_file)['initial_positions']}"/>
         <ros2_control name="${name}" type="system">
             <hardware>
-                <!-- By default, set up controllers for simulation. This won't work on real hardware -->
-                <plugin>mock_components/GenericSystem</plugin>
+                <xacro:if value="${use_real_hardware}">
+                    <plugin>tl_hardware/TLHardwareInterface</plugin>
+                    <param name="joint_states_topic">/joint_states</param>
+                    <param name="servoj_topic">/tl_driver/set_servoj_pos</param>
+                    <param name="open_servoj_service">/tl_driver/open_servoj</param>
+                    <param name="close_servoj_service">/tl_driver/close_servoj</param>
+                    <param name="state_timeout_sec">1.0</param>
+                </xacro:if>
+                <xacro:unless value="${use_real_hardware}">
+                    <plugin>mock_components/GenericSystem</plugin>
+                </xacro:unless>
             </hardware>
             <joint name="joint1">

File: src/tl_moveit2_config/tl_tcb605l_config/config/tl_tcb605l.urdf.xacro (robot description, xacro)
@@ -2,8 +2,9 @@
 <robot xmlns:xacro="http://www.ros.org/wiki/xacro" name="tl_tcb605l">
     <xacro:arg name="initial_positions_file" default="initial_positions.yaml" />
+    <xacro:arg name="use_real_hardware" default="false" />
     <!-- Import tl_tcb605l urdf file -->
     <xacro:include filename="$(find tl_description)/urdf/tcb605l.urdf" />
     <!-- Import control_xacro -->
     <xacro:include filename="tl_tcb605l.ros2_control.xacro" />
-    <xacro:tl_tcb605l_ros2_control name="FakeSystem" initial_positions_file="$(arg initial_positions_file)"/>
+    <xacro:tl_tcb605l_ros2_control name="FakeSystem" initial_positions_file="$(arg initial_positions_file)" use_real_hardware="$(arg use_real_hardware)"/>
 </robot>

File: src/tl_moveit2_config/tl_tcb605lv_config/config/tl_tcb605lv.ros2_control.xacro (robot description, xacro)
@@ -1,10 +1,19 @@
 <?xml version="1.0"?>
 <robot xmlns:xacro="http://www.ros.org/wiki/xacro">
-    <xacro:macro name="tl_tcb605lv_ros2_control" params="name initial_positions_file">
+    <xacro:macro name="tl_tcb605lv_ros2_control" params="name initial_positions_file use_real_hardware:=false">
         <xacro:property name="initial_positions" value="${xacro.load_yaml(initial_positions_file)['initial_positions']}"/>
         <ros2_control name="${name}" type="system">
             <hardware>
-                <!-- By default, set up controllers for simulation. This won't work on real hardware -->
-                <plugin>mock_components/GenericSystem</plugin>
+                <xacro:if value="${use_real_hardware}">
+                    <plugin>tl_hardware/TLHardwareInterface</plugin>
+                    <param name="joint_states_topic">/joint_states</param>
+                    <param name="servoj_topic">/tl_driver/set_servoj_pos</param>
+                    <param name="open_servoj_service">/tl_driver/open_servoj</param>
+                    <param name="close_servoj_service">/tl_driver/close_servoj</param>
+                    <param name="state_timeout_sec">1.0</param>
+                </xacro:if>
+                <xacro:unless value="${use_real_hardware}">
+                    <plugin>mock_components/GenericSystem</plugin>
+                </xacro:unless>
             </hardware>
             <joint name="joint1">

File: src/tl_moveit2_config/tl_tcb605lv_config/config/tl_tcb605lv.urdf.xacro (robot description, xacro)
@@ -2,8 +2,9 @@
 <robot xmlns:xacro="http://www.ros.org/wiki/xacro" name="tl_tcb605lv">
     <xacro:arg name="initial_positions_file" default="initial_positions.yaml" />
+    <xacro:arg name="use_real_hardware" default="false" />
     <!-- Import tl_tcb605lv urdf file -->
     <xacro:include filename="$(find tl_description)/urdf/tcb605lv.urdf" />
     <!-- Import control_xacro -->
     <xacro:include filename="tl_tcb605lv.ros2_control.xacro" />
-    <xacro:tl_tcb605lv_ros2_control name="FakeSystem" initial_positions_file="$(arg initial_positions_file)"/>
+    <xacro:tl_tcb605lv_ros2_control name="FakeSystem" initial_positions_file="$(arg initial_positions_file)" use_real_hardware="$(arg use_real_hardware)"/>
 </robot>

File: src/tl_moveit2_config/tl_tcb605v_config/config/tl_tcb605v.ros2_control.xacro (robot description, xacro)
@@ -1,10 +1,19 @@
 <?xml version="1.0"?>
 <robot xmlns:xacro="http://www.ros.org/wiki/xacro">
-    <xacro:macro name="tl_tcb605v_ros2_control" params="name initial_positions_file">
+    <xacro:macro name="tl_tcb605v_ros2_control" params="name initial_positions_file use_real_hardware:=false">
         <xacro:property name="initial_positions" value="${xacro.load_yaml(initial_positions_file)['initial_positions']}"/>
         <ros2_control name="${name}" type="system">
             <hardware>
-                <!-- By default, set up controllers for simulation. This won't work on real hardware -->
-                <plugin>mock_components/GenericSystem</plugin>
+                <xacro:if value="${use_real_hardware}">
+                    <plugin>tl_hardware/TLHardwareInterface</plugin>
+                    <param name="joint_states_topic">/joint_states</param>
+                    <param name="servoj_topic">/tl_driver/set_servoj_pos</param>
+                    <param name="open_servoj_service">/tl_driver/open_servoj</param>
+                    <param name="close_servoj_service">/tl_driver/close_servoj</param>
+                    <param name="state_timeout_sec">1.0</param>
+                </xacro:if>
+                <xacro:unless value="${use_real_hardware}">
+                    <plugin>mock_components/GenericSystem</plugin>
+                </xacro:unless>
             </hardware>
             <joint name="joint1">

File: src/tl_moveit2_config/tl_tcb605v_config/config/tl_tcb605v.urdf.xacro (robot description, xacro)
@@ -2,8 +2,9 @@
 <robot xmlns:xacro="http://www.ros.org/wiki/xacro" name="tl_tcb605v">
     <xacro:arg name="initial_positions_file" default="initial_positions.yaml" />
+    <xacro:arg name="use_real_hardware" default="false" />
     <!-- Import tl_tcb605v urdf file -->
     <xacro:include filename="$(find tl_description)/urdf/tcb605v.urdf" />
     <!-- Import control_xacro -->
     <xacro:include filename="tl_tcb605v.ros2_control.xacro" />
-    <xacro:tl_tcb605v_ros2_control name="FakeSystem" initial_positions_file="$(arg initial_positions_file)"/>
+    <xacro:tl_tcb605v_ros2_control name="FakeSystem" initial_positions_file="$(arg initial_positions_file)" use_real_hardware="$(arg use_real_hardware)"/>
 </robot>

File: src/tl_moveit2_config/tl_tcb610_config/config/tl_tcb610.ros2_control.xacro (robot description, xacro)
@@ -1,10 +1,19 @@
 <?xml version="1.0"?>
 <robot xmlns:xacro="http://www.ros.org/wiki/xacro">
-    <xacro:macro name="tl_tcb610_ros2_control" params="name initial_positions_file">
+    <xacro:macro name="tl_tcb610_ros2_control" params="name initial_positions_file use_real_hardware:=false">
         <xacro:property name="initial_positions" value="${xacro.load_yaml(initial_positions_file)['initial_positions']}"/>
         <ros2_control name="${name}" type="system">
             <hardware>
-                <!-- By default, set up controllers for simulation. This won't work on real hardware -->
-                <plugin>mock_components/GenericSystem</plugin>
+                <xacro:if value="${use_real_hardware}">
+                    <plugin>tl_hardware/TLHardwareInterface</plugin>
+                    <param name="joint_states_topic">/joint_states</param>
+                    <param name="servoj_topic">/tl_driver/set_servoj_pos</param>
+                    <param name="open_servoj_service">/tl_driver/open_servoj</param>
+                    <param name="close_servoj_service">/tl_driver/close_servoj</param>
+                    <param name="state_timeout_sec">1.0</param>
+                </xacro:if>
+                <xacro:unless value="${use_real_hardware}">
+                    <plugin>mock_components/GenericSystem</plugin>
+                </xacro:unless>
             </hardware>
             <joint name="joint1">

File: src/tl_moveit2_config/tl_tcb610_config/config/tl_tcb610.urdf.xacro (robot description, xacro)
@@ -2,8 +2,9 @@
 <robot xmlns:xacro="http://www.ros.org/wiki/xacro" name="tl_tcb610">
     <xacro:arg name="initial_positions_file" default="initial_positions.yaml" />
+    <xacro:arg name="use_real_hardware" default="false" />
     <!-- Import tl_tcb610 urdf file -->
     <xacro:include filename="$(find tl_description)/urdf/tcb610.urdf" />
     <!-- Import control_xacro -->
     <xacro:include filename="tl_tcb610.ros2_control.xacro" />
-    <xacro:tl_tcb610_ros2_control name="FakeSystem" initial_positions_file="$(arg initial_positions_file)"/>
+    <xacro:tl_tcb610_ros2_control name="FakeSystem" initial_positions_file="$(arg initial_positions_file)" use_real_hardware="$(arg use_real_hardware)"/>
 </robot>

File: src/tl_moveit2_config/tl_tcb610v_config/config/tl_tcb610v.ros2_control.xacro (robot description, xacro)
@@ -1,10 +1,19 @@
 <?xml version="1.0"?>
 <robot xmlns:xacro="http://www.ros.org/wiki/xacro">
-    <xacro:macro name="tl_tcb610v_ros2_control" params="name initial_positions_file">
+    <xacro:macro name="tl_tcb610v_ros2_control" params="name initial_positions_file use_real_hardware:=false">
         <xacro:property name="initial_positions" value="${xacro.load_yaml(initial_positions_file)['initial_positions']}"/>
         <ros2_control name="${name}" type="system">
             <hardware>
-                <!-- By default, set up controllers for simulation. This won't work on real hardware -->
-                <plugin>mock_components/GenericSystem</plugin>
+                <xacro:if value="${use_real_hardware}">
+                    <plugin>tl_hardware/TLHardwareInterface</plugin>
+                    <param name="joint_states_topic">/joint_states</param>
+                    <param name="servoj_topic">/tl_driver/set_servoj_pos</param>
+                    <param name="open_servoj_service">/tl_driver/open_servoj</param>
+                    <param name="close_servoj_service">/tl_driver/close_servoj</param>
+                    <param name="state_timeout_sec">1.0</param>
+                </xacro:if>
+                <xacro:unless value="${use_real_hardware}">
+                    <plugin>mock_components/GenericSystem</plugin>
+                </xacro:unless>
             </hardware>
             <joint name="joint1">

File: src/tl_moveit2_config/tl_tcb610v_config/config/tl_tcb610v.urdf.xacro (robot description, xacro)
@@ -2,8 +2,9 @@
 <robot xmlns:xacro="http://www.ros.org/wiki/xacro" name="tl_tcb610v">
     <xacro:arg name="initial_positions_file" default="initial_positions.yaml" />
+    <xacro:arg name="use_real_hardware" default="false" />
     <!-- Import tl_tcb610v urdf file -->
     <xacro:include filename="$(find tl_description)/urdf/tcb610v.urdf" />
     <!-- Import control_xacro -->
     <xacro:include filename="tl_tcb610v.ros2_control.xacro" />
-    <xacro:tl_tcb610v_ros2_control name="FakeSystem" initial_positions_file="$(arg initial_positions_file)"/>
+    <xacro:tl_tcb610v_ros2_control name="FakeSystem" initial_positions_file="$(arg initial_positions_file)" use_real_hardware="$(arg use_real_hardware)"/>
 </robot>

File: src/tl_moveit2_config/tl_tcb705_config/config/tl_tcb705.ros2_control.xacro (robot description, xacro)
@@ -1,10 +1,19 @@
 <?xml version="1.0"?>
 <robot xmlns:xacro="http://www.ros.org/wiki/xacro">
-    <xacro:macro name="tl_tcb705_ros2_control" params="name initial_positions_file">
+    <xacro:macro name="tl_tcb705_ros2_control" params="name initial_positions_file use_real_hardware:=false">
         <xacro:property name="initial_positions" value="${xacro.load_yaml(initial_positions_file)['initial_positions']}"/>
         <ros2_control name="${name}" type="system">
             <hardware>
-                <!-- By default, set up controllers for simulation. This won't work on real hardware -->
-                <plugin>mock_components/GenericSystem</plugin>
+                <xacro:if value="${use_real_hardware}">
+                    <plugin>tl_hardware/TLHardwareInterface</plugin>
+                    <param name="joint_states_topic">/joint_states</param>
+                    <param name="servoj_topic">/tl_driver/set_servoj_pos</param>
+                    <param name="open_servoj_service">/tl_driver/open_servoj</param>
+                    <param name="close_servoj_service">/tl_driver/close_servoj</param>
+                    <param name="state_timeout_sec">1.0</param>
+                </xacro:if>
+                <xacro:unless value="${use_real_hardware}">
+                    <plugin>mock_components/GenericSystem</plugin>
+                </xacro:unless>
             </hardware>
             <joint name="joint1">

File: src/tl_moveit2_config/tl_tcb705_config/config/tl_tcb705.urdf.xacro (robot description, xacro)
@@ -2,8 +2,9 @@
 <robot xmlns:xacro="http://www.ros.org/wiki/xacro" name="tl_tcb705">
     <xacro:arg name="initial_positions_file" default="initial_positions.yaml" />
+    <xacro:arg name="use_real_hardware" default="false" />
     <!-- Import tl_tcb705 urdf file -->
     <xacro:include filename="$(find tl_description)/urdf/tcb705.urdf" />
     <!-- Import control_xacro -->
     <xacro:include filename="tl_tcb705.ros2_control.xacro" />
-    <xacro:tl_tcb705_ros2_control name="FakeSystem" initial_positions_file="$(arg initial_positions_file)"/>
+    <xacro:tl_tcb705_ros2_control name="FakeSystem" initial_positions_file="$(arg initial_positions_file)" use_real_hardware="$(arg use_real_hardware)"/>
 </robot>

File: src/tl_moveit2_config/tl_tcb705f_config/config/tl_tcb705f.ros2_control.xacro (robot description, xacro)
@@ -1,10 +1,19 @@
 <?xml version="1.0"?>
 <robot xmlns:xacro="http://www.ros.org/wiki/xacro">
-    <xacro:macro name="tl_tcb705f_ros2_control" params="name initial_positions_file">
+    <xacro:macro name="tl_tcb705f_ros2_control" params="name initial_positions_file use_real_hardware:=false">
         <xacro:property name="initial_positions" value="${xacro.load_yaml(initial_positions_file)['initial_positions']}"/>
         <ros2_control name="${name}" type="system">
             <hardware>
-                <!-- By default, set up controllers for simulation. This won't work on real hardware -->
-                <plugin>mock_components/GenericSystem</plugin>
+                <xacro:if value="${use_real_hardware}">
+                    <plugin>tl_hardware/TLHardwareInterface</plugin>
+                    <param name="joint_states_topic">/joint_states</param>
+                    <param name="servoj_topic">/tl_driver/set_servoj_pos</param>
+                    <param name="open_servoj_service">/tl_driver/open_servoj</param>
+                    <param name="close_servoj_service">/tl_driver/close_servoj</param>
+                    <param name="state_timeout_sec">1.0</param>
+                </xacro:if>
+                <xacro:unless value="${use_real_hardware}">
+                    <plugin>mock_components/GenericSystem</plugin>
+                </xacro:unless>
             </hardware>
             <joint name="joint1">

File: src/tl_moveit2_config/tl_tcb705f_config/config/tl_tcb705f.urdf.xacro (robot description, xacro)
@@ -2,8 +2,9 @@
 <robot xmlns:xacro="http://www.ros.org/wiki/xacro" name="tl_tcb705f">
     <xacro:arg name="initial_positions_file" default="initial_positions.yaml" />
+    <xacro:arg name="use_real_hardware" default="false" />
     <!-- Import tl_tcb705f urdf file -->
     <xacro:include filename="$(find tl_description)/urdf/tcb705f.urdf" />
     <!-- Import control_xacro -->
     <xacro:include filename="tl_tcb705f.ros2_control.xacro" />
-    <xacro:tl_tcb705f_ros2_control name="FakeSystem" initial_positions_file="$(arg initial_positions_file)"/>
+    <xacro:tl_tcb705f_ros2_control name="FakeSystem" initial_positions_file="$(arg initial_positions_file)" use_real_hardware="$(arg use_real_hardware)"/>
 </robot>

File: src/tl_moveit2_config/tl_tcb705l_config/config/tl_tcb705l.ros2_control.xacro (robot description, xacro)
@@ -1,10 +1,19 @@
 <?xml version="1.0"?>
 <robot xmlns:xacro="http://www.ros.org/wiki/xacro">
-    <xacro:macro name="tl_tcb705l_ros2_control" params="name initial_positions_file">
+    <xacro:macro name="tl_tcb705l_ros2_control" params="name initial_positions_file use_real_hardware:=false">
         <xacro:property name="initial_positions" value="${xacro.load_yaml(initial_positions_file)['initial_positions']}"/>
         <ros2_control name="${name}" type="system">
             <hardware>
-                <!-- By default, set up controllers for simulation. This won't work on real hardware -->
-                <plugin>mock_components/GenericSystem</plugin>
+                <xacro:if value="${use_real_hardware}">
+                    <plugin>tl_hardware/TLHardwareInterface</plugin>
+                    <param name="joint_states_topic">/joint_states</param>
+                    <param name="servoj_topic">/tl_driver/set_servoj_pos</param>
+                    <param name="open_servoj_service">/tl_driver/open_servoj</param>
+                    <param name="close_servoj_service">/tl_driver/close_servoj</param>
+                    <param name="state_timeout_sec">1.0</param>
+                </xacro:if>
+                <xacro:unless value="${use_real_hardware}">
+                    <plugin>mock_components/GenericSystem</plugin>
+                </xacro:unless>
             </hardware>
             <joint name="joint1">

File: src/tl_moveit2_config/tl_tcb705l_config/config/tl_tcb705l.urdf.xacro (robot description, xacro)
@@ -2,8 +2,9 @@
 <robot xmlns:xacro="http://www.ros.org/wiki/xacro" name="tl_tcb705l">
     <xacro:arg name="initial_positions_file" default="initial_positions.yaml" />
+    <xacro:arg name="use_real_hardware" default="false" />
     <!-- Import tl_tcb705l urdf file -->
     <xacro:include filename="$(find tl_description)/urdf/tcb705l.urdf" />
     <!-- Import control_xacro -->
     <xacro:include filename="tl_tcb705l.ros2_control.xacro" />
-    <xacro:tl_tcb705l_ros2_control name="FakeSystem" initial_positions_file="$(arg initial_positions_file)"/>
+    <xacro:tl_tcb705l_ros2_control name="FakeSystem" initial_positions_file="$(arg initial_positions_file)" use_real_hardware="$(arg use_real_hardware)"/>
 </robot>

File: src/tl_moveit2_config/tl_tcb705lv_config/config/tl_tcb705lv.ros2_control.xacro (robot description, xacro)
@@ -1,10 +1,19 @@
 <?xml version="1.0"?>
 <robot xmlns:xacro="http://www.ros.org/wiki/xacro">
-    <xacro:macro name="tl_tcb705lv_ros2_control" params="name initial_positions_file">
+    <xacro:macro name="tl_tcb705lv_ros2_control" params="name initial_positions_file use_real_hardware:=false">
         <xacro:property name="initial_positions" value="${xacro.load_yaml(initial_positions_file)['initial_positions']}"/>
         <ros2_control name="${name}" type="system">
             <hardware>
-                <!-- By default, set up controllers for simulation. This won't work on real hardware -->
-                <plugin>mock_components/GenericSystem</plugin>
+                <xacro:if value="${use_real_hardware}">
+                    <plugin>tl_hardware/TLHardwareInterface</plugin>
+                    <param name="joint_states_topic">/joint_states</param>
+                    <param name="servoj_topic">/tl_driver/set_servoj_pos</param>
+                    <param name="open_servoj_service">/tl_driver/open_servoj</param>
+                    <param name="close_servoj_service">/tl_driver/close_servoj</param>
+                    <param name="state_timeout_sec">1.0</param>
+                </xacro:if>
+                <xacro:unless value="${use_real_hardware}">
+                    <plugin>mock_components/GenericSystem</plugin>
+                </xacro:unless>
             </hardware>
             <joint name="joint1">
