Commit message: feat:moveit2控制真实机械臂完成所有型号适配

File: src/tl_moveit2_config/tl_tcb705lv_config/config/tl_tcb705lv.urdf.xacro (robot description, xacro)
@@ -2,8 +2,9 @@
 <robot xmlns:xacro="http://www.ros.org/wiki/xacro" name="tl_tcb705lv">
     <xacro:arg name="initial_positions_file" default="initial_positions.yaml" />
+    <xacro:arg name="use_real_hardware" default="false" />
     <!-- Import tl_tcb705lv urdf file -->
     <xacro:include filename="$(find tl_description)/urdf/tcb705lv.urdf" />
     <!-- Import control_xacro -->
     <xacro:include filename="tl_tcb705lv.ros2_control.xacro" />
-    <xacro:tl_tcb705lv_ros2_control name="FakeSystem" initial_positions_file="$(arg initial_positions_file)"/>
+    <xacro:tl_tcb705lv_ros2_control name="FakeSystem" initial_positions_file="$(arg initial_positions_file)" use_real_hardware="$(arg use_real_hardware)"/>
 </robot>
